File: DEMI_Buffer.kicad_sch (KiCad schematic)
At the start: 19 parts, among them J1 SJ2-35853A-SMT-TR, J2 ASMPR45-1X2-RK, Q1 IRLML2060, U2 L78L05_SOT89, U3 SN74LVC1G14DBV

Commit message: Cleaned up the repo a bit
Cleaned up the repo a bit
Other:
- note removed: "TEST PLAN: *** HAVE A THINK BEFORE RUNNING*** Test 0: Action: Apply 12V to J2 Verify: Power rails and default states Status: Pass Test 1: Action: Connect and only power-on IC705 Verify: Measure 5V Bus for leakage and Q1 Vgs for turn-on (expect none) Status: Pass - Voltage across R4=0.00V, indicates very weak pull-up on the IC-705. Test 2: Action: Connect and only power-on DEMI Verify: Measure 5V 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"
Changed lines of the file:
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@@
     (effects (font (size 2.54 2.54)) (justify left bottom))
-  )
-  (text "TEST PLAN:\n*** HAVE A THINK BEFORE RUNNING***\nTest 0:\n    Action: Apply 12V to J2\n    Verify: Power rails and default states\n    Status: Pass\nTest 1:\n    Action: Connect and only power-on IC705\n    Verify: Measure 5V Bus for leakage and Q1 Vgs for turn-on (expect none)\n    Status: Pass - Voltage across R4=0.00V, indicates very weak pull-up on the IC-705.\nTest 2:\n    Action: Connect and only power-on DEMI\n    Verify: Measure 5V Bus (expect good), U3 input and output voltage, Q1 Vgs, Resistance across PTT and GND, Voltage across RELAY + and -\nTest 3:\n    Action: Install Dummy Load on DEMI, Connect and only power-on DEMI and toggle the SEND input with a PSU or function generator\n    Verify: Measure expected behavior at U3, Q1 voltage and current, and RELAY + and -\nTest 4:\n    Action: Install Dummy Load on DEMI, Connect and power-on IC-705 and DEMI. Use SEND and IF cable (do a microwave safety check first and use minimum or no power)\n    Verify: Functionality"
-    (at 21.59 165.1 0)
-    (effects (font (size 1.27 1.27)) (justify left bottom))
   )
   (text "DEMI Voltage: 10-15.5V" (at 190.5 67.31 0)
